File: pcbs/sweep-pro/sweep-pro-left/sweep-pro-left.kicad_pcb (KiCad board)
At the start: 2 copper layers, 115 x 86.7 mm, 48 parts, among them SW1 SW_PUSH-kbd, SW10 SW_PUSH-kbd, SW11 SW_PUSH-kbd, SW12 SW_PUSH-kbd, SW13 SW_PUSH-kbd, SW14 SW_PUSH-kbd, SW15 SW_PUSH-kbd, SW16 SW_PUSH-kbd, SW17 SW_PUSH-kbd, SW2 SW_PUSH-kbd, SW3 SW_PUSH-kbd, SW4 SW_PUSH-kbd, SW5 SW_PUSH-kbd, SW6 SW_PUSH-kbd, SW7 SW_PUSH-kbd, SW8 SW_PUSH-kbd, SW9 SW_PUSH-kbd, U1 ProMicro-kbd

Commit message: backup
Parts:
- removed Bat_extra1: Conn_Battery_pluggable, mylib:Molex_Panelmate_53780-0270_1x02-1MP_P1.25mm_Horizontal
- added J1: Conn_01x04_Female, mylib:pogopin_1x4, F.Cu at (202.5, 53.0)
- added J2: Conn_01x04_Female, mylib:pogopin_1x4, F.Cu at (200.0, 53.0)
- added J3: expantion1, mylib:pogopin_1x4, F.Cu at (178.6, 100.3)
- Bat_main1: footprint mylib:Battery_pads_reversible -> mylib:Molex_Panelmate_53780-0270_1x02-1MP_P1.25mm_Horizontal
- D1, D10, D11, D12, D13, D14, D15, D16, D17, D2, D3, D4, D5, D6, D7, D8, D9: footprint mylib:Diode_SOD-123_reversible -> mylib:Diode
- D18: footprint mylib:Diode_SOD-123_reversible -> mylib:Diode; moved to B.Cu
- U1: footprint mylib:ProMacroLite_BackMount_Partial -> mylib:ProMacroLite_Partial
- moved Bat_main1 43.7 mm to (167.0, 99.0), turned to 130 degrees
- moved D18 4.25 mm to (199.2, 91.3), turned to -5 degrees
- moved SW_Power1 0.08 mm to (209.7, 96.9)
Connections:
- Encoder1 pad S1: col4 -> col3
- U1 pad 1: bsy -> 0.06
- U1 pad 10: encoder_a -> bsy
- U1 pad 11: sw_encoder -> row4
- U1 pad 12: row4 -> encoder_b
- U1 pad 16: col5 -> col1
- U1 pad 17: col4 -> col2
- U1 pad 19: col2 -> col4
- U1 pad 2: rst -> 0.08
- U1 pad 20: col1 -> col5
- U1 pad 21: VCC -> unconnected-(U1-Pad21)
- U1 pad 29: 3.3V -> VCC
- U1 pad 31: 1.04 -> encoder_a
- U1 pad 5: din -> rst
- U1 pad 6: clk -> din
- U1 pad 7: dc -> clk
- U1 pad 8: cs -> dc
- U1 pad 9: encoder_b -> cs
Routing:
- net col1: track 33.4 -> 175.3 mm, vias 0 -> 4
- net col2: track 34.0 -> 157.8 mm, vias 0 -> 4
- net col3: track 34.9 -> 131.6 mm, vias 2 -> 4
- net row4: track 20.7 -> 101.4 mm, vias 0 -> 4
- net VRaw: track 0.00 -> 68.2 mm
- net VBus: track 0.00 -> 55.1 mm
- net rst: track 0.00 -> 50.6 mm
- net bsy: track 0.00 -> 43.9 mm, vias 0 -> 4
- net VBat: track 0.00 -> 41.6 mm
- net row3: track 87.2 -> 125.3 mm
- net clk: track 0.00 -> 35.9 mm
- net col4: track 69.0 -> 104.7 mm, vias 0 -> 4
- net din: track 0.00 -> 33.8 mm
- net reset: track 33.0 -> 65.8 mm, vias 2 -> 0
- net GND: track 137.7 -> 110.9 mm, vias 41 -> 29
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
Commit message: sweepro-left intial finished version
Routing:
- net GND: vias 29 -> 40
