File: pcbs/sweep-pro/sweep-pro-left/sweep-pro-left.kicad_sch (KiCad schematic)
At the start: 41 parts, among them SW1 SW_PUSH-kbd, SW10 SW_PUSH-kbd, SW11 SW_PUSH-kbd, SW12 SW_PUSH-kbd, SW13 SW_PUSH-kbd, SW14 SW_PUSH-kbd, SW15 SW_PUSH-kbd, SW16 SW_PUSH-kbd, SW17 SW_PUSH-kbd, SW2 SW_PUSH-kbd, SW3 SW_PUSH-kbd, SW4 SW_PUSH-kbd, SW5 SW_PUSH-kbd, SW6 SW_PUSH-kbd, SW7 SW_PUSH-kbd, SW8 SW_PUSH-kbd, SW9 SW_PUSH-kbd, U1 ProMicro-kbd

Commit message: backup
Parts:
- added D18: 1N4148W, mylib:Diode_SOD-123_reversible, symbol mysymbol:1N4148W
- added H1, H2, H3, H4: MountingHole, MountingHole:MountingHole_2.2mm_M2_ISO7380_Pad_TopBottom, symbol Mechanical:MountingHole
- added H5: MountingHole, MountingHole:MountingHole_3.2mm_M3_DIN965, symbol Mechanical:MountingHole
- added WirelessCharger1: Conn_01x02_Female, mylib:VBus_pad_reversible, symbol Connector:Conn_01x02_Female
- D1, D10, D11, D12, D13, D14, D15, D16, D17, D2, D3, D4, D5, D6, D7, D8, D9: footprint Diode_SMD:D_SOD-123 -> mylib:Diode_SOD-123_reversible; symbol Diode:1N4148W -> mysymbol:1N4148W
- Display1: footprint mylib:Conn_EPD_Jumper -> mylib:Conn_EPD
- SW1, SW10, SW11, SW14, SW15, SW16, SW17, SW2, SW3, SW4, SW5, SW6, SW7, SW8, SW9: footprint mylib:Kailh_Choc_reversible -> mylib:Kailh_Choc_Hotplug
- SW_Power1: value SW_Battery_kbd -> SW_Battery-kbd; footprint mylib:Power_reversible -> mylib:SW_BSI10; symbol mysymbol:SW_Battery_kbd -> mysymbol:SW_Battery-kbd
- U1: footprint mylib:ProMicro_Jumpers -> mylib:ProMacroLite_BackMount_Partial; symbol mysymbol:ProMicro-kbd -> mysymbol:ProMacro-Lite-Partial
Connections:
- net GND: now also U1.28 (gnd), WirelessCharger1.gnd (GND); no longer Encoder1.S2
- net col4: now also Encoder1.S1
- net encoder_a: now also U1.10 (E6); no longer U1.9 (D7)
- net encoder_b: now also U1.9 (D7); no longer U1.10 (E6)
- net row4: now also D18.1 (K)
- net sw_encoder: no longer Encoder1.S1
- new net: D18.2 (A), Encoder1.S2
- new net 0.05: U1.30
- new net 1.04: U1.31
- new net 3.3V: U1.29 (3.3V)
- new net VBus: U1.25 (vbus), WirelessCharger1.+5V
- no-connect marks 0 -> 1

Commit message: backup
Parts:
- removed Bat_extra1: Conn_Battery_pluggable, mylib:Battery_connector_lim_reversible, symbol mysymbol:Conn_Battery_pluggable
- added J1, J2: Conn_01x04_Female, mylib:pogopin_1x4, symbol Connector:Conn_01x04_Female
- added J3: expantion1, mylib:pogopin_1x4, symbol Connector:Conn_01x04_Female
- Bat_main1: footprint mylib:Battery_pads_reversible -> mylib:Molex_Panelmate_53780-0270_1x02-1MP_P1.25mm_Horizontal
- D1, D10, D11, D12, D13, D14, D15, D16, D17, D18, D2, D3, D4, D5, D6, D7, D8, D9: footprint mylib:Diode_SOD-123_reversible -> mylib:Diode
Connections:
- net 1.04 is gone; now on net encoder_a: U1.31
- net 3.3V is gone; now on net VCC: U1.29 (3.3V)
- net sw_encoder is gone; now on net row4: U1.11 (B4)
- net 0.05: now also J1.3 (Pin_3)
- net GND: now also J2.4 (Pin_4)
- net VBus: now also WirelessCharger1.vbus (VBUS); no longer WirelessCharger1.+5V
- net VCC: now also J1.4 (Pin_4); no longer U1.21 (VCC)
- net bsy: now also U1.10 (E6), J2.3 (Pin_3); no longer U1.1 (TX)
- net clk: now also U1.7 (D4), J2.2 (Pin_2); no longer U1.6 (SCL)
- net col1: now also U1.16 (B1), J3.2 (Pin_2); no longer U1.20 (F4)
- net col2: now also U1.17 (F7), J3.1 (Pin_1); no longer U1.19 (F5)
- net col3: now also Encoder1.S1
- net col4: now also U1.19 (F5); no longer Encoder1.S1, U1.17 (F7)
- net col5: now also U1.20 (F4); no longer U1.16 (B1)
- net cs: now also U1.9 (D7); no longer U1.8 (C6)
- net dc: now also U1.8 (C6); no longer U1.7 (D4)
- net din: now also U1.6 (SCL), J2.1 (Pin_1); no longer U1.5 (SDA)
- net encoder_a: no longer U1.10 (E6)
- net encoder_b: now also U1.12 (B5); no longer U1.9 (D7)
- net row4: now also J3.3 (Pin_3), J3.4 (Pin_4); no longer U1.12 (B5)
- net rst: now also U1.5 (SDA); no longer U1.2 (RX)
- new net 0.06: J1.1 (Pin_1), U1.1 (TX)
- new net 0.08: J1.2 (Pin_2), U1.2 (RX)
- no-connect marks 1 -> 2
Other:
- note added: "expansion port (expose 6 hi-frq gpio, vcc and gnd)"
- note added: "expantion port (opitional two more switches in row4)"
- moved on the sheet: Bat_main1, D18, Encoder1, H4, H5, SW_Reset1, WirelessCharger1

Commit message: backup
Parts:
- H1, H2, H3, H4: footprint MountingHole:MountingHole_2.2mm_M2_ISO7380_Pad_TopBottom -> MountingHole:MountingHole_3.2mm_M3_DIN965
- SW12, SW13: footprint mylib:Kailh_Choc_reversible -> mylib:Kailh_Choc_Hotplug
Changed lines of the file:
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@@
     (property "Reference" "SW14" (id 0) (at 207.01 73.66 0))
     (property "Value" "SW_PUSH-kbd" (id 1) (at 207.01 76.2 0))
-    (property "Footprint" "mylib:Kailh_Choc_Hotplug" (id 2) (at 207.01 81.28 0))
+    (property "Footprint" "mylib:Kailh_Choc_Hotplug" (id 2) (at 207.01 81.28 0)
+      (effects (font (size 1.27 1.27)) hide)
+    )
     (property "Datasheet" "" (id 3) (at 207.01 81.28 0))
     (pin "1")
@@
     (property "Reference" "SW13" (id 0) (at 181.61 73.66 0))
     (property "Value" "SW_PUSH-kbd" (id 1) (at 181.61 76.2 0))
-    (property "Footprint" "mylib:Kailh_Choc_reversible" (id 2) (at 181.61 81.28 0)
+    (property "Footprint" "mylib:Kailh_Choc_Hotplug" (id 2) (at 181.61 81.28 0)
       (effects (font (size 1.27 1.27)) hide)
     )
@@
     (property "Reference" "SW12" (id 0) (at 156.21 73.66 0))
     (property "Value" "SW_PUSH-kbd" (id 1) (at 156.21 76.2 0))
-    (property "Footprint" "mylib:Kailh_Choc_reversible" (id 2) (at 156.21 81.28 0)
+    (property "Footprint" "mylib:Kailh_Choc_Hotplug" (id 2) (at 156.21 81.28 0)
       (effects (font (size 1.27 1.27)) hide)
     )
@@
       (effects (font (size 1.27 1.27)) (justify left))
     )
-    (property "Footprint" "MountingHole:MountingHole_2.2mm_M2_ISO7380_Pad_TopBottom" (id 2) (at 67.31 176.53 0)
+    (property "Footprint" "MountingHole:MountingHole_3.2mm_M3_DIN965" (id 2) (at 67.31 176.53 0)
       (effects (font (size 1.27 1.27)) hide)
     )
@@
       (effects (font (size 1.27 1.27)) (justify left))
     )
-    (property "Footprint" "MountingHole:MountingHole_2.2mm_M2_ISO7380_Pad_TopBottom" (id 2) (at 22.86 187.96 0)
+    (property "Footprint" "MountingHole:MountingHole_3.2mm_M3_DIN965" (id 2) (at 22.86 187.96 0)
       (effects (font (size 1.27 1.27)) hide)
     )
@@
       (effects (font (size 1.27 1.27)) (justify left))
     )
-    (property "Footprint" "MountingHole:MountingHole_2.2mm_M2_ISO7380_Pad_TopBottom" (id 2) (at 44.45 176.53 0)
+    (property "Footprint" "MountingHole:MountingHole_3.2mm_M3_DIN965" (id 2) (at 44.45 176.53 0)
       (effects (font (size 1.27 1.27)) hide)
     )
@@
       (effects (font (size 1.27 1.27)) (justify left))
     )
-    (property "Footprint" "MountingHole:MountingHole_2.2mm_M2_ISO7380_Pad_TopBottom" (id 2) (at 22.86 176.53 0)
+    (property "Footprint" "MountingHole:MountingHole_3.2mm_M3_DIN965" (id 2) (at 22.86 176.53 0)
       (effects (font (size 1.27 1.27)) hide)
     )
@@
     )
     (path "/fc087110-f130-4c78-bc07-c99d7b1b6356"
-      (reference "H1") (unit 1) (value "MountingHole") (footprint "MountingHole:MountingHole_2.2mm_M2_ISO7380_Pad_TopBottom")
+      (reference "H1") (unit 1) (value "MountingHole") (footprint "MountingHole:MountingHole_3.2mm_M3_DIN965")
     )
     (path "/ad9b87a9-429e-4aea-bc42-5ce1607773cd"
-      (reference "H2") (unit 1) (value "MountingHole") (footprint "MountingHole:MountingHole_2.2mm_M2_ISO7380_Pad_TopBottom")
+      (reference "H2") (unit 1) (value "MountingHole") (footprint "MountingHole:MountingHole_3.2mm_M3_DIN965")
     )
     (path "/50ecd970-c920-4563-901d-56351b4c513a"
-      (reference "H3") (unit 1) (value "MountingHole") (footprint "MountingHole:MountingHole_2.2mm_M2_ISO7380_Pad_TopBottom")
+      (reference "H3") (unit 1) (value "MountingHole") (footprint "MountingHole:MountingHole_3.2mm_M3_DIN965")
     )
     (path "/84009376-d132-496d-bc3c-c9b99bc8a0ad"
-      (reference "H4") (unit 1) (value "MountingHole") (footprint "MountingHole:MountingHole_2.2mm_M2_ISO7380_Pad_TopBottom")
+      (reference "H4") (unit 1) (value "MountingHole") (footprint "MountingHole:MountingHole_3.2mm_M3_DIN965")
     )
     (path "/9dd58876-f968-4cd0-b2ad-422f53c41329"
@@
     )
     (path "/42c9a293-e5eb-4d22-a688-16bbe175b2d6"
-      (reference "SW12") (unit 1) (value "SW_PUSH-kbd") (footprint "mylib:Kailh_Choc_reversible")
+      (reference "SW12") (unit 1) (value "SW_PUSH-kbd") (footprint "mylib:Kailh_Choc_Hotplug")
     )
     (path "/39617f4c-c890-48ec-aab9-807080b3cf1a"
-      (reference "SW13") (unit 1) (value "SW_PUSH-kbd") (footprint "mylib:Kailh_Choc_reversible")
+      (reference "SW13") (unit 1) (value "SW_PUSH-kbd") (footprint "mylib:Kailh_Choc_Hotplug")
     )
     (path "/10c88ae6-b3e0-47ce-a55c-5111940f5c50"
