File: pcbs/corne-pro-nrfmicro/left/left.kicad_sch (KiCad schematic)
At the start: 53 parts, among them SW1 SW_PUSH-kbd, SW10 SW_PUSH-kbd, SW11 SW_PUSH-kbd, SW12 SW_PUSH-kbd, SW13 SW_PUSH-kbd, SW14 SW_PUSH-kbd, SW15 SW_PUSH-kbd, SW16 SW_PUSH-kbd, SW17 SW_PUSH-kbd, SW18 SW_PUSH-kbd, SW19 SW_PUSH-kbd, SW2 SW_PUSH-kbd, SW20 SW_PUSH-kbd, SW21 SW_PUSH-kbd, SW3 SW_PUSH-kbd, SW4 SW_PUSH-kbd, SW5 SW_PUSH-kbd, SW6 SW_PUSH-kbd, SW7 SW_PUSH-kbd, SW8 SW_PUSH-kbd, SW9 SW_PUSH-kbd, U1 ProMicro-kbd

Commit message: add gerber zip file
Parts:
- Bat_backup1: footprint mylib:Molex_Panelmate_53780-0270_1x02-1MP_P1.25mm_Horizontal -> Connector_JST:JST_ACH_BM02B-ACHSS-GAN-ETF_1x02-1MP_P1.20mm_Vertical
Changed lines of the file:
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@@
       (effects (font (size 1.27 1.27)) (justify left) hide)
     )
-    (property "Footprint" "mylib:Molex_Panelmate_53780-0270_1x02-1MP_P1.25mm_Horizontal" (id 2) (at 55.88 129.54 0)
+    (property "Footprint" "Connector_JST:JST_ACH_BM02B-ACHSS-GAN-ETF_1x02-1MP_P1.20mm_Vertical" (id 2) (at 55.88 129.54 0)
       (effects (font (size 1.27 1.27)) hide)
     )
@@
   (symbol (lib_id "power:GND") (at 50.8 134.62 0) (unit 1)
     (in_bom yes) (on_board yes) (fields_autoplaced)
-    (property "Reference" "#PWR?" (id 0) (at 50.8 140.97 0)
+    (property "Reference" "#PWR0101" (id 0) (at 50.8 140.97 0)
       (effects (font (size 1.27 1.27)) hide)
     )
@@
     )
     (path "/de2781d3-8dd3-47b8-a4a7-9c68b110e628"
-      (reference "#PWR?") (unit 1) (value "GND") (footprint "")
+      (reference "#PWR0101") (unit 1) (value "GND") (footprint "")
     )
     (path "/0a48f02f-76ac-4f18-962a-1aa9912cfba0"
-      (reference "Bat_backup1") (unit 1) (value "Conn_Battery_solderable") (footprint "mylib:Molex_Panelmate_53780-0270_1x02-1MP_P1.25mm_Horizontal")
+      (reference "Bat_backup1") (unit 1) (value "Conn_Battery_solderable") (footprint "Connector_JST:JST_ACH_BM02B-ACHSS-GAN-ETF_1x02-1MP_P1.20mm_Vertical")
     )
     (path "/67451d5d-77ee-4a05-8359-b8d0301e96b4"
