File: pcbs/sweep-pro-ce/sweep-pro-ce.kicad_pcb (KiCad board)
At the start: 2 copper layers, 115 x 86.7 mm, 50 parts, among them SW1 SW_PUSH-kbd, SW10 SW_PUSH-kbd, SW11 SW_PUSH-kbd, SW12 SW_PUSH-kbd, SW13 SW_PUSH-kbd, SW14 SW_PUSH-kbd, SW15 SW_PUSH-kbd, SW16 SW_PUSH-kbd, SW17 SW_PUSH-kbd, SW2 SW_PUSH-kbd, SW3 SW_PUSH-kbd, SW4 SW_PUSH-kbd, SW5 SW_PUSH-kbd, SW6 SW_PUSH-kbd, SW7 SW_PUSH-kbd, SW8 SW_PUSH-kbd, SW9 SW_PUSH-kbd, U1 ProMicro-kbd

Commit message: backup
Parts:
- H1, H2, H3, H4, H5: footprint MountingHole:MountingHole_3.2mm_M3_DIN965 -> mylib:MountingHole_3.2mm_M3_DIN965
