File: pcbs/sweep-pro/sweep-pro-trackball-right/encoder.kicad_sch (KiCad schematic)
At the start: 2 parts

Commit message: init version with integrated trackball in thumb position
Parts:
- Encoder1: footprint mylib:RollerEncoder_Panasonic_EVQWGD001 -> mylib:Panasonic_EVQWGD001_Latest
Changed lines of the file:
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@@
       (effects (font (size 1.27 1.27)) hide)
     )
-    (property "Footprint" "mylib:RollerEncoder_Panasonic_EVQWGD001" (id 2) (at 142.494 97.79 0)
+    (property "Footprint" "mylib:Panasonic_EVQWGD001_Latest" (id 2) (at 142.494 97.79 0)
       (effects (font (size 1.27 1.27)) hide)
     )
