File: pcbs/sweep-pro/sweep-pro-trackball-right/keyboard.kicad_sch (KiCad schematic)
At the start: 36 parts, among them J1 expantion1, J2 Conn_01x04_Female, SW1 SW_PUSH-kbd, SW10 SW_PUSH-kbd, SW11 SW_PUSH-kbd, SW12 SW_PUSH-kbd, SW13 SW_PUSH-kbd, SW14 SW_PUSH-kbd, SW15 SW_PUSH-kbd, SW16 SW_PUSH-kbd, SW17 SW_PUSH-kbd, SW2 SW_PUSH-kbd, SW3 SW_PUSH-kbd, SW4 SW_PUSH-kbd, SW5 SW_PUSH-kbd, SW6 SW_PUSH-kbd, SW7 SW_PUSH-kbd, SW8 SW_PUSH-kbd, SW9 SW_PUSH-kbd

Commit message: init version with integrated trackball in thumb position
Parts:
- J2: footprint (none) -> mylib:pogopin_1x4
Changed lines of the file:
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@@
       (effects (font (size 1.27 1.27)) hide)
     )
-    (property "Footprint" "" (id 2) (at 115.57 186.182 0)
+    (property "Footprint" "mylib:pogopin_1x4" (id 2) (at 115.57 186.182 0)
       (effects (font (size 1.27 1.27)) hide)
     )
