File: pcbs/blade/right/blade-right.kicad_pcb (KiCad board)
At the start: 2 copper layers, 133 x 86.7 mm, 106 parts, among them J1 expantion1, J10 Conn_01x07, J11 Conn_01x04_Female, J12 USB-C USB 2.0 MC-372, J16 Conn_01x03_Male, J3 Conn_01x07, J5 Conn_01x05, J9 Conn_Display_general, Q1 AO3407, Q2 AO3407, SW1 SW_PUSH-kbd, SW10 SW_PUSH-kbd, SW11 SW_PUSH-kbd, SW12 SW_PUSH-kbd, SW14 SW_PUSH-kbd, SW15 SW_PUSH-kbd, SW16 SW_PUSH-kbd, SW17 SW_PUSH-kbd, SW18 SW_PUSH-kbd, SW19 SW_PUSH-kbd, SW2 SW_PUSH-kbd, SW20 SW_PUSH-kbd, SW3 SW_PUSH-kbd, SW4 SW_PUSH-kbd, SW5 SW_PUSH-kbd, SW6 SW_PUSH-kbd, SW7 SW_PUSH-kbd, SW8 SW_PUSH-kbd, SW9 SW_PUSH-kbd, U1 E73-2G4M08S1C, U2 SRV05-4, U3 XC6220B331MR-G, U4 MAX17048, U5 TP4054, U6 PMW3610, U7 MCP1700-1802E-TT, U8 CAP1203, X1 32.768 kHz

Commit message: backup
Parts:
- moved D21 103.9 mm to (165.4, 141.4)
- moved Encoder1 103.9 mm to (163.4, 139.9)
- moved J5 103.9 mm to (163.4, 139.9)
- moved C12 23.5 mm to (125.1, 134.8), turned to 0 degrees
- moved C13 20.0 mm to (122.0, 134.8), turned to 180 degrees
- moved C5 16.4 mm to (118.4, 134.9), turned to 180 degrees
- moved C11 15.6 mm to (120.9, 149.1), turned to 0 degrees
- moved U7 14.3 mm to (105.5, 135.5), turned to -90 degrees
- moved C6 14.0 mm to (108.8, 134.3), turned to 0 degrees
- moved C8 14.0 mm to (115.2, 134.9), turned to 0 degrees
- moved C7 12.9 mm to (112.0, 134.9), turned to 180 degrees
- moved C10 11.9 mm to (108.8, 135.8), turned to 0 degrees
- moved R13 11.6 mm to (117.6, 149.1), turned to 0 degrees
- moved JP1 10.00 mm to (105.2, 147.7), turned to -90 degrees
- moved C9 9.16 mm to (106.7, 139.3), turned to 90 degrees
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